File: eagle/sanfrancisco_barometer_rev_C.sch (EAGLE design)
At the start: 39 parts, among them IC1 PIC18F2580, IC2 MPL115A1, IC3 MCP2551SN, IC4 LM2575S, IC5 LM2931M, J2 A00-108-220-450, Q1 10 MHz

Commit message: Changed component symbols
Connections:
- new net N$8: C11.2, IC1.RA4/T0CKIN
- net VCC: no longer C11.2, IC1.RA4/T0CKIN
Other:
- note added: "C"
- note removed: "B"
Changed lines of the file:
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@@
 <part name="PAD1" library="wirepad" deviceset="1,6/0,8" device=""/>
 <part name="PAD2" library="wirepad" deviceset="1,6/0,8" device=""/>
-<part name="P+5" library="SUPPLY1" deviceset="VCC" device=""/>
 <part name="IC5" library="v-reg-3" deviceset="LM2931" device="M"/>
 <part name="P+10" library="SUPPLY1" deviceset="VCC" device=""/>
@@
 <text x="200.66" y="177.8" size="1.778" layer="91">ALPS SKHH</text>
 <text x="200.66" y="175.26" size="1.778" layer="91">Horizontal type</text>
-<text x="378.46" y="7.62" size="1.778" layer="91">B</text>
+<text x="378.46" y="7.62" size="1.778" layer="91">C</text>
 <text x="289.56" y="27.94" size="5.08" layer="91">San Franscisco</text>
 <text x="365.76" y="25.4" size="1.778" layer="91">http://www.vscp.org</text>
@@
 <instance part="PAD1" gate="P" x="248.92" y="246.38"/>
 <instance part="PAD2" gate="P" x="248.92" y="238.76"/>
-<instance part="P+5" gate="VCC" x="15.24" y="220.98"/>
 <instance part="IC5" gate="A" x="99.06" y="114.3"/>
 <instance part="P+10" gate="VCC" x="81.28" y="129.54"/>
@@
 </segment>
 <segment>
-<wire x1="15.24" y1="203.2" x2="15.24" y2="198.12" width="0.1524" layer="91"/>
-<wire x1="81.28" y1="203.2" x2="15.24" y2="203.2" width="0.1524" layer="91"/>
-<pinref part="C11" gate="G$1" pin="2"/>
-<pinref part="IC1" gate="G$1" pin="RA4/T0CKIN"/>
-<pinref part="P+5" gate="VCC" pin="VCC"/>
-<wire x1="15.24" y1="218.44" x2="15.24" y2="203.2" width="0.1524" layer="91"/>
-<junction x="15.24" y="203.2"/>
-</segment>
-<segment>
 <pinref part="P+10" gate="VCC" pin="VCC"/>
 <pinref part="C13" gate="G$1" pin="2"/>
@@
 </segment>
 </net>
+<net name="N$8" class="0">
+<segment>
+<wire x1="15.24" y1="203.2" x2="15.24" y2="198.12" width="0.1524" layer="91"/>
+<wire x1="81.28" y1="203.2" x2="15.24" y2="203.2" width="0.1524" layer="91"/>
+<pinref part="C11" gate="G$1" pin="2"/>
+<pinref part="IC1" gate="G$1" pin="RA4/T0CKIN"/>
+</segment>
+</net>
